Commit message: Add setup script for zsh and log files for build events
- Created a new zsh setup script to extend the environment with other prefix paths.
- Added COLCON_IGNORE file to the log directory.
- Generated log files for build events and logger output for the pathbot_simulation package.

File: install/pathbot_description/share/pathbot_description/urdf/robot.gazebo.xacro (robot description, xacro)
@@ -1 +1,111 @@
-/home/hornet/Desktop/pathfollowingbot/src/pathbot_description/urdf/robot.gazebo.xacro
+<?xml version="1.0"?>
+<robot name="robo_robot" xmlns:xacro="https://www.ros.org/wiki/xacro">
+<xacro:include filename ="$(find pathbot_description)/urdf/robot.xacro"/>
+<!-- <gazebo>
+    <model>
+        <canonical_link>body_link</canonical_link>
+    </model>
+</gazebo> -->
+<gazebo reference = "body_link">
+    <mu1>0.2</mu1>
+    <mu2>0.2</mu2>
+    <material>Gazebo/Red</material>
+</gazebo>
+<gazebo reference = "wheel1_link">
+    <mu1>1.0</mu1>
+    <mu2>1.0</mu2>
+    <material>Gazebo/Yellow</material>
+</gazebo>
+<gazebo reference = "wheel2_link">
+    <mu1>1.0</mu1>
+    <mu2>1.0</mu2>
+    <material>Gazebo/Yellow</material>
+</gazebo>
+<gazebo reference = "wheel3_link">
+    <mu1>1.0</mu1>
+    <mu2>1.0</mu2>
+    <material>Gazebo/Yellow</material>
+</gazebo
+>
+<gazebo reference = "wheel4_link">
+    <mu1>1.0</mu1>
+    <mu2>1.0</mu2>
+    <material>Gazebo/Yellow</material>
+</gazebo>
+<!-- <gazebo reference = "caster_link">
+    <mu1>0.00002</mu1>
+    <mu2>0.00002</mu2>
+    <material>Gazebo/Blue</material>
+</gazebo> -->
+<gazebo>
+    <plugin filename = "libgz-sim-diff-drive-system.so" name="gz::sim::systems::DiffDrive">
+        <left_joint>wheel1_joint</left_joint>
+        <left_joint>wheel3_joint</left_joint>
+        <right_joint>wheel2_joint</right_joint>
+        <right_joint>wheel4_joint</right_joint>
+        <wheel_separation>${2*s4}</wheel_separation>
+        <wheel_radius>${radius}</wheel_radius>
+        <max_wheel_torque>150</max_wheel_torque>
+        <max_wheel_acceleration>20.0</max_wheel_acceleration>
+        <topic>/cmd_vel</topic>
+        <tf_topic>/tf</tf_topic>
+        <odom_topic>/odom</odom_topic>
+        <frame_id>odom</frame_id>
+        <child_frame_id>body_footprint</child_frame_id>
+        <odom_publisher_frequency>30</odom_publisher_frequency>
+    </plugin>
+    <plugin filename="libgz-sim-joint-state-publisher-system.so" name="gz::sim::systems::JointStatePublisher">
+        <topic>/joint_states</topic>
+        <joint_name>wheel1_joint</joint_name>
+        <joint_name>wheel2_joint</joint_name>
+        <joint_name>wheel3_joint</joint_name>
+        <joint_name>wheel4_joint</joint_name>
+    </plugin>
+</gazebo>
+<!--
+sensor is world pulggin not a robot pluggin
+<gazebo>
+    <plugin filename="libgz-sim-sensors-system.so"
+            name="gz::sim::systems::Sensors">
+        <render_engine>ogre2</render_engine>
+    </plugin>
+</gazebo> -->
+<!-- LiDAR sensor -->
+<gazebo reference="lidar_link">
+<!-- get to gpu lidar if it nromlly starts to work also cpu lidar that is normal lidar is not supportd in ros gazebo 8-->
+    <sensor name="gpu_lidar" type="gpu_lidar">
+        <!-- <ray>
+            <collision>
+                <ignore_entity>robo_robot</ignore_entity>
+            </collision>
+        </ray> -->
+        <!-- as it is directely attached to lidar link -->
+    <pose>0 0 0 0 0 0</pose>
+    <topic>scan</topic>
+    <update_rate>10</update_rate>
+    <lidar>
+        <scan>
+            <horizontal>
+                <samples>720</samples>
+                <resolution>1</resolution>
+                <min_angle>-3.14159</min_angle>
+                <max_angle>3.14159</max_angle>
+            </horizontal>
+        </scan>
+        <range>
+            <min>0.1</min>
+            <max>12.0</max>
+            <resolution>0.01</resolution>
+        </range>
+        <noise>
+            <type>gaussian</type>
+            <mean>0.0</mean>
+            <stddev>0.001</stddev>
+        </noise>
+    </lidar>
+    <always_on>true</always_on>
+    <!-- only for testing turning it of -->
+    <visualize>true</visualize>
+    </sensor>
+</gazebo>
+</robot>

File: install/pathbot_description/share/pathbot_description/urdf/robot.xacro (robot description, xacro)
@@ -1 +1,274 @@
-/home/hornet/Desktop/pathfollowingbot/src/pathbot_description/urdf/robot.xacro
+<?xml version='1.0'?>
+<robot name = "robo_robot" xmlns:xacro="http://www.ros.org/wiki/xacro">
+<!-- define constants -->
+<xacro:property name = "ohm" value ="3.14159"/>
+<!-- BODY LINK DIMENSIONS  -->
+<!-- units used in meters -->
+<xacro:property name = "body_length"
+   value ="1.0"/>
+<xacro:property name = "body_height"
+   value ="0.30"/>
+<xacro:property name = "body_width"
+   value ="0.60"/>
+<!-- WHEEL DIMENSIONS  AND CASTOR DIMENSIONS -->
+<!-- RADIUS -->
+<xacro:property name = "radius"
+   value = "0.15"/>
+<!-- WIDTH  WHEEL -->
+<xacro:property name ="width"
+   value ="0.10"/>
+<xacro:property name ="wheel_z_location"
+   value ="-0.1"/>
+<!-- other dimensions -->
+<xacro:property name = "s1"
+   value = "${body_height/2 + radius}"/>
+<xacro:property name = "s2"
+   value ="${radius*2}"/>
+<xacro:property name = "s3"
+   value = "${radius*2}"/>
+<xacro:property name = "s4"
+   value ="${body_width/2 + width/2}"/>
+<!-- MASS NAD INERTIA -->
+<!-- DENSITY -->
+<!-- BODY LINK -->
+<xacro:property name = "body_link"
+   value = "500.0"/>
+<!-- WHEEL LINK -->
+<xacro:property name = "wheel_link"
+   value = "500.0"/>
+<!-- CASTOR LINK
+<xacro:property name = "castor_link"
+   value = "500.0"/> -->
+<!-- MASS -->
+<!-- BODY LINK MASS -->
+<xacro:property name = "body_mass"
+   value = "${body_link*body_length*body_width*body_height}"/>
+<!-- WHEEL LINK MASS -->
+<xacro:property name = "wheel_mass"
+   value = "${wheel_link*ohm*radius*radius*width}"/>
+<!-- CASTOR LINK MASS
+<xacro:property name = "castor_mass"
+   value = "${castor_link*(4/3)*ohm*radius*radius*radius}"/> -->
+<!--MOMENT OF INERTIA -->
+<!-- BODY LINK MOMENT OF INERTIA -->
+<xacro:property name = "Ix_body"
+   value = "${(1/12)*body_mass*(body_height*body_height + body_width*body_width)}" />
+<xacro:property name = "Iy_body"
+   value = "${(1/12)*body_mass*(body_length*body_length + body_width*body_width)}" />
+<xacro:property name = "Iz_body"
+   value = "${(1/12)*body_mass*(body_length*body_length + body_height*body_height)}" />
+<!-- WHEEL LINK MOMENT OF INERTIA -->
+<xacro:property name="Ix_wheel"
+   value="${(1/12)*wheel_mass*(3*radius*radius + width*width)}"/>
+<xacro:property name="Iy_wheel"
+   value="${(1/2)*wheel_mass*radius*radius}"/>
+<xacro:property name="Iz_wheel"
+   value="${(1/12)*wheel_mass*(3*radius*radius + width*width)}"/>
+<!-- CASTOR LINK MOMENT OF INERTIA
+<xacro:property name = "Ix_castor"
+   value = "${(2/5)*castor_mass*radius*radius}" />
+<xacro:property name = "Iy_castor"
+   value = "${(2/5)*castor_mass*radius*radius}" />
+<xacro:property name = "Iz_castor"
+   value = "${(2/5)*castor_mass*radius*radius}" /> -->
+<!-- complete inertial system of the body -->
+<!-- FILE THAT INCLUDES GAZEBO OPTIONS AND MOTION CONTROLS-->
+<!-- THE BASIC COORDINATE SYSTEM IS CENTERED AT THE GEOMETRIC CENTER OF THE BODY LINK -->
+<!-- dummy link for gazebo
+<link name="dummy">
+</link>
+<joint name="dummy_joint" type="fixed">
+   <parent link="dummy"/>
+   <child link="body_link"/>
+</joint> -->
+<!-- BODY LINK -->
+<xacro:macro name = "body_link_macro">
+   <inertial>
+   <origin xyz = " 0 0 ${radius}" rpy = "0 0 0"/>
+   <mass value = "${body_mass}"/>
+   <inertia ixx ="${Ix_body}" ixy = "0.0" ixz ="0.0" iyy ="${Iy_body}" iyz = "0.0" izz= "${Iz_body}"/>
+   </inertial>
+</xacro:macro>
+<!-- WHEEL LINK -->
+<xacro:macro name = "wheel_link_macro">
+   <inertial>
+   <origin xyz = "0 0 0" rpy = "0 0 0"/>
+   <mass value = "${wheel_mass}"/>
+   <inertia ixx ="${Ix_wheel}" ixy="0.0" ixz="0.0" iyy="${Iy_wheel}" iyz ="0.0" izz="${Iz_wheel}"/>
+   </inertial>
+</xacro:macro>
+<!-- CASTOR LINK
+<xacro:macro name = "castor_link_macro">
+   <inertial>
+   <origin xyz = "0 0 0" rpy = "1.57095 0 0"/>
+   <mass value = "${castor_mass}"/>
+   <inertia ixx = "${Ix_castor}" ixy= "0.0" ixz="0.0" iyy="${Iy_castor}" iyz="0.0" izz= "${Iz_castor}"/>
+   </inertial>
+</xacro:macro> -->
+<!-- INERTFACE FOR COMTROLS -->
+<!-- FICTOUS LINK  -->
+<!-- DEFINING LINKS ANDS JOINTS -->
+<link name  = "body_footprint"></link>
+<joint name = "body_link_joint" type = "fixed">
+   <parent link = "body_footprint"/>
+   <child link = "body_link"/>
+</joint>
+<!-- BODY LINK OF ROBOT -->
+<link name = "body_link">
+   <visual>
+      <geometry>
+         <box size = "${body_length} ${body_width} ${body_height}"/>
+      </geometry>
+      <origin xyz="0 0 ${radius}" rpy = "0 0 0"/>
+   </visual>
+   <collision>
+      <geometry>
+         <box size = "${body_length} ${body_width} ${body_height}"/>
+      </geometry>
+      <origin xyz="0 0 ${radius}" rpy = "0 0 0"/>
+   </collision>
+   <xacro:body_link_macro/>
+</link>
+<!-- WHEEL JOINT -->
+<joint name="wheel1_joint" type ="continuous">
+   <parent link = "body_link"/>
+   <child link = "wheel1_link"/>
+   <origin xyz= " ${-s2} ${-s4} 0" rpy="0 0 0"/>
+   <axis xyz= "0 1 0"/>
+   <limit effort = "100000" velocity= "10"/>
+   <dynamics damping ="1.0" friction ="1.0"/>
+</joint>
+<link name = "wheel1_link">
+   <visual>
+      <geometry>
+         <cylinder length = "${width}" radius = "${radius}"/>
+      </geometry>
+      <origin xyz = "0 0 0" rpy = "1.570795 0 0"/>
+   </visual>
+   <collision>
+      <geometry>
+         <cylinder length = "${width}" radius = "${radius}"/>
+      </geometry>
+      <origin xyz = "0 0 0" rpy = "1.570795 0 0"/>
+   </collision>
+   <xacro:wheel_link_macro/>
+</link>
+<joint name="wheel2_joint" type ="continuous">
+   <parent link = "body_link"/>
+   <child link = "wheel2_link"/>
+   <origin xyz= " ${-s2} ${s4} 0" rpy="0 0 0"/>
+   <axis xyz= "0 1 0"/>
+   <limit effort = "100000" velocity= "10"/>
+   <dynamics damping ="1.0" friction ="1.0"/>
+</joint>
+<link name ="wheel2_link">
+   <visual>
+      <geometry>
+         <cylinder length = "${width}" radius = "${radius}"/>
+      </geometry>
+      <origin xyz = "0 0 0" rpy = "1.570795 0 0"/>
+   </visual>
+   <collision>
+      <geometry>
+         <cylinder length = "${width}" radius = "${radius}"/>
+      </geometry>
+      <origin xyz = "0 0 0" rpy = "1.570795 0 0"/>
+   </collision>
+   <xacro:wheel_link_macro/>
+</link>
+<joint name="wheel3_joint" type="continuous">
+   <parent link="body_link"/>
+   <child link="wheel3_link"/>
+   <origin xyz="${s2} ${-s4} 0" rpy="0 0 0"/>
+   <axis xyz="0 1 0"/>
+   <limit effort="100000" velocity="10"/>
+   <dynamics damping="1.0" friction="1.0"/>
+</joint>
+<link name="wheel3_link">
+   <visual>
+      <geometry>
+         <cylinder length="${width}" radius="${radius}"/>
+      </geometry>
+      <origin xyz="0 0 0" rpy="1.570795 0 0"/>
+   </visual>
+   <collision>
+      <geometry>
+         <cylinder length="${width}" radius="${radius}"/>
+      </geometry>
+      <origin xyz="0 0 0" rpy="1.570795 0 0"/>
+   </collision>
+   <xacro:wheel_link_macro/>
+</link>
+<joint name="wheel4_joint" type="continuous">
+   <parent link="body_link"/>
+   <child link="wheel4_link"/>
+   <origin xyz="${s2} ${s4} 0" rpy="0 0 0"/>
+   <axis xyz="0 1 0"/>
+   <limit effort="100000" velocity="10"/>
+   <dynamics damping="1.0" friction="1.0"/>
+</joint>
+<link name="wheel4_link">
+   <visual>
+      <geometry>
+         <cylinder length="${width}" radius="${radius}"/>
+      </geometry>
+      <origin xyz="0 0 0" rpy="1.570795 0 0"/>
+   </visual>
+   <collision>
+      <geometry>
+         <cylinder length="${width}" radius="${radius}"/>
+      </geometry>
+      <origin xyz="0 0 0" rpy="1.570795 0 0"/>
+   </collision>
+   <xacro:wheel_link_macro/>
+</link>
+<!-- CASTOR JOINT
+<joint name="caster_joint" type ="continuous">
+   <parent link = "body_link"/>
+   <child link = "caster_link"/>
+   <origin xyz= " ${body_length/2 - radius} 0 0" rpy="1.570795 0 0"/>
+   <axis xyz= "0 1 0"/>
+   <limit effort = "100000" velocity= "10"/>
+   <dynamics damping ="1.0" friction ="1.0"/>
+</joint>
+<link name = "caster_link">
+   <visual>
+      <geometry>
+         <sphere radius = "${radius}"/>
+      </geometry>
+      <origin xyz = "0 0 0" rpy = "1.570795 0 0"/>
+   </visual>
+   <collision>
+      <geometry>
+         <sphere radius = "${radius}"/>
+      </geometry>
+      <origin xyz = "0 0 0" rpy = "1.570795 0 0"/>
+   </collision>
+   <xacro:castor_link_macro/>
+</link>   -->
+<!-- LIDAR -->
+<joint name = "lidar_joint" type = "fixed">
+   <origin xyz="0 0 0.35" rpy="0 0 0"/>
+   <parent link="body_link"/>
+   <child link="lidar_link"/>
+</joint>
+<link name="lidar_link">
+   <visual>
+   <origin xyz="0 0 0" rpy="0 0 0"/>
+      <geometry>
+         <cylinder length ="0.1" radius="0.1"/>
+      </geometry>
+   </visual>
+   <!-- <collision name ="collision">
+      <origin xyz="0 0 0" rpy="0 0 0"/>
+      <geometry>
+         <cylinder length ="0.1" radius="0.1"/>
+      </geometry>
+   </collision> -->
+   <inertial>
+      <mass value="1e-6"/>
+      <origin xyz="0 0 0" rpy="0 0 0"/>
+      <inertia ixx="1e-6" ixy="0" ixz="0" iyy="1e-6" iyz="0" izz="1e-6"/>
+   </inertial>
+</link>
+</robot>

File: src/pathbot_description/urdf/robot.xacro (robot description, xacro)
@@ -87,5 +87,5 @@
    <origin xyz = " 0 0 ${radius}" rpy = "0 0 0"/>
    <mass value = "${body_mass}"/>
-   <inertia ixx ="${Ix_body}" ixy = "0.0" ixz ="0.0" iyy ="${Iz_body}" iyz = "0.0" izz= "${Iy_body}"/>
+   <inertia ixx ="${Ix_body}" ixy = "0.0" ixz ="0.0" iyy ="${Iy_body}" iyz = "0.0" izz= "${Iz_body}"/>
    </inertial>
 </xacro:macro>
@@ -252,5 +252,4 @@
    <parent link="body_link"/>
    <child link="lidar_link"/>
-   <axis xyz="0 1 0" rpy="0 0 0"/>
 </joint>
 <link name="lidar_link">

Commit message: edited the  xacro file to correct the  rotation of the wheels of left and right hand side

File: install/pathbot_description/share/pathbot_description/urdf/robot.gazebo.xacro (robot description, xacro)
@@ -2,4 +2,10 @@
 <robot name="robo_robot" xmlns:xacro="https://www.ros.org/wiki/xacro">
 <xacro:include filename ="$(find pathbot_description)/urdf/robot.xacro"/>
+<!-- Skid-steer scrub correction for the DiffDrive odometry. The four fixed
+     wheels scrub sideways when turning, so the effective track is wider than
+     the geometric 2*s4 = 0.70 m. Measured against Gazebo ground truth: odom
+     over-reported yaw by ~2.1x at 1.0, then under-reported by 9% at 2.10.
+     Converged value below; see the calibration procedure in COMMANDS.md. -->
+<xacro:property name="track_correction" value="1.91"/>
 <!-- <gazebo>
     <model>
@@ -26,6 +32,5 @@
     <mu2>1.0</mu2>
     <material>Gazebo/Yellow</material>
-</gazebo
->
+</gazebo>
 <gazebo reference = "wheel4_link">
     <mu1>1.0</mu1>
@@ -40,18 +45,25 @@
 <gazebo>
     <plugin filename = "libgz-sim-diff-drive-system.so" name="gz::sim::systems::DiffDrive">
-        <left_joint>wheel1_joint</left_joint>
-        <left_joint>wheel3_joint</left_joint>
-        <right_joint>wheel2_joint</right_joint>
-        <right_joint>wheel4_joint</right_joint>
-        <wheel_separation>${2*s4}</wheel_separation>
+        <!-- +y is LEFT (REP-103). wheel2/wheel4 sit at y=+s4, wheel1/wheel3 at
+             y=-s4. Getting this backwards inverts the sign of odometry yaw and
+             destroys SLAM on every turn. -->
+        <left_joint>wheel2_joint</left_joint>
+        <left_joint>wheel4_joint</left_joint>
+        <right_joint>wheel1_joint</right_joint>
+        <right_joint>wheel3_joint</right_joint>
+        <!-- 4-wheel skid-steer: the wheels scrub sideways when turning, so the
+             effective track is wider than the geometric 2*s4. Calibrated
+             against Gazebo ground truth - see COMMANDS.md. -->
+        <wheel_separation>${2*s4*track_correction}</wheel_separation>
         <wheel_radius>${radius}</wheel_radius>
-        <max_wheel_torque>150</max_wheel_torque>
-        <max_wheel_acceleration>20.0</max_wheel_acceleration>
         <topic>/cmd_vel</topic>
         <tf_topic>/tf</tf_topic>
         <odom_topic>/odom</odom_topic>
+        <!-- Required. Without it the odom frame becomes "robo_robot/odom",
+             which breaks the odom->body_footprint TF chain and makes
+             slam_toolbox drop every scan ("queue is full"). -->
         <frame_id>odom</frame_id>
         <child_frame_id>body_footprint</child_frame_id>
-        <odom_publisher_frequency>30</odom_publisher_frequency>
+        <odom_publish_frequency>30</odom_publish_frequency>
     </plugin>
     <plugin filename="libgz-sim-joint-state-publisher-system.so" name="gz::sim::systems::JointStatePublisher">
